File: KiCad/rf_switch_filter/rf_switch_filter.kicad_pcb (KiCad board)
At the start: 2 copper layers, 22 parts, among them J1 Screw_Terminal_01x04, J10 FILTER_OUT, J5 5V From SDR, J9 ANT, U17 BPF-A355, U3 SKY13588-460LF, U4 SKY13588-460LF, U5 SN74AVC2T244DQER, U6 MIC5365-1.8YC5-TR, U7 MIC5365-3.3YC5-TR

Commit message: Fix up RF switch project
Laid out schematic to be more legible, added screw terminals from wiring
diagram, changed GND symbols, changed labels to be global labels, and
added project libraries
Connections:
- net /RFS_GND renamed /GND
- net /RFSwitchFilter/5V_IN renamed /RFSwitchFilter/5V
- net /RFSwitchFilter/VDD_REF renamed /RFSwitchFilter/VDD
