File: KiCad/smd_filter/smd_filter.kicad_sch (KiCad schematic)
At the start: 0 parts

Commit message: Port over smd_filter
Parts:
- added J11, J15: ANT, Library:CONN_142-0711-821_CIN, symbol Connector:Conn_Coaxial
- added U15: BPF-A1340+, RF_Mini-Circuits:Mini-Circuits_HQ1157, symbol RF_Filter:BPF-A355
Connections:
- new net GND: J11.2 (Ext), J15.2 (Ext), U15.10 (GND), U15.11 (GND), U15.12 (GND), U15.13 (GND), U15.14 (GND), U15.2 (GND), U15.3 (GND), U15.4 (GND), U15.5 (GND), U15.6 (GND), U15.7 (GND), U15.9 (GND)
- new net SIGNAL IN: J11.1 (In), U15.1 (IN)
- new net SIGNAL OUT: J15.1 (In), U15.8 (OUT)
